File: pcb-for-nano-s2/flight-controller.kicad_pcb (KiCad board)
At the start: 4 copper layers, 24 x 33 mm, 59 parts, among them J1 BM03B-SRSS-TBLFSN, J2 BM03B-SRSS-TBLFSN, J3 BM03B-SRSS-TBLFSN, J4 Conn_01x02, J5 Conn_ARM_JTAG_SWD_10, J6 Conn_01x02, Q1 Q_NMOS_GSD, Q2 Q_NMOS_GSD, U1 STM32G4A1KEU6, U2 ZOE-M8Q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

Commit message: change PCB design to six layers
Routing:
- added copper zone on In3.Cu, net +3V3
- added copper zone on In1.Cu, net GND
- added copper zone on In4.Cu, net GND
- removed copper zone on In1.Cu, net +3V3
Other:
- copper layers 4 -> 6
Changed lines of the file:
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@@
 (kicad_pcb (version 20221018) (generator pcbnew)
   (general
-    (thickness 0.98)
+    (thickness 0.585)
   )
   (paper "A4")
@@
     (1 "In1.Cu" signal)
     (2 "In2.Cu" signal)
+    (3 "In3.Cu" signal)
+    (4 "In4.Cu" signal)
     (31 "B.Cu" signal)
     (32 "B.Adhes" user "B.Adhesive")
@@
       (layer "F.Mask" (type "Top Solder Mask") (color "Green") (thickness 0.01))
       (layer "F.Cu" (type "copper") (thickness 0.035))
-      (layer "dielectric 1" (type "core") (thickness 0.11) (material "FR4") (epsilon_r 4.3) (loss_tangent 0.02))
+      (layer "dielectric 1" (type "prepreg") (thickness 0.071) (material "FR4") (epsilon_r 4.3) (loss_tangent 0.02))
       (layer "In1.Cu" (type "copper") (thickness 0.035))
-      (layer "dielectric 2" (type "prepreg") (thickness 0.6) (material "FR4") (epsilon_r 4.3) (loss_tangent 0.02))
+      (layer "dielectric 2" (type "core") (thickness 0.071) (material "FR4") (epsilon_r 4.3) (loss_tangent 0.02))
       (layer "In2.Cu" (type "copper") (thickness 0.035))
-      (layer "dielectric 3" (type "core") (thickness 0.11) (material "FR4") (epsilon_r 4.3) (loss_tangent 0.02))
+      (layer "dielectric 3" (type "prepreg") (thickness 0.071) (material "FR4") (epsilon_r 4.3) (loss_tangent 0.02))
+      (layer "In3.Cu" (type "copper") (thickness 0.035))
+      (layer "dielectric 4" (type "core") (thickness 0.071) (material "FR4") (epsilon_r 4.5) (loss_tangent 0.02))
+      (layer "In4.Cu" (type "copper") (thickness 0.035))
+      (layer "dielectric 5" (type "prepreg") (thickness 0.071) (material "FR4") (epsilon_r 4.5) (loss_tangent 0.02))
       (layer "B.Cu" (type "copper") (thickness 0.035))
       (layer "B.Mask" (type "Bottom Solder Mask") (color "Green") (thickness 0.01))
       (layer "B.Paste" (type "Bottom Solder Paste"))
       (layer "B.SilkS" (type "Bottom Silk Screen"))
-      (copper_finish "ENIG")
+      (copper_finish "None")
       (dielectric_constraints no)
     )
@@
     (fp_circle (center 0 0) (end 0.4 0)
       (stroke (width 0.1) (type solid)) (fill none) (layer "F.Fab"))
-    (pad "1" thru_hole roundrect (at 0 0 90) (size 1 1) (drill 0.6) (layers "*.Mask" "F.Cu" "In1.Cu" "In2.Cu" "B.Cu") (roundrect_rratio 0.15625)
+    (pad "1" thru_hole roundrect (at 0 0 90) (size 1 1) (drill 0.6) (layers "*.Cu" "*.Mask") (roundrect_rratio 0.15625)
       (net 17 "Net-(RADIO1-Pin_1)") (pinfunction "Pin_1") (pintype "passive"))
     (model "${KICAD6_3DMODEL_DIR}/Connector_Wire.3dshapes/SolderWire-0.1sqmm_1x01_D0.4mm_OD1mm.wrl"
@@
     (fp_line (start 1.6 0.6) (end 1.6 -0.6)
       (stroke (width 0.127) (type solid)) (layer "F.Fab"))
-    (pad "" np_thru_hole circle (at 0 0 90) (size 1.75 1.75) (drill 1.75) (layers "F&B.Cu" "*.Mask"))
+    (pad "" np_thru_hole circle (at 0 0 90) (size 1.75 1.75) (drill 1.75) (layers "*.Cu" "*.Mask"))
     (pad "1" smd roundrect (at -1.65 -0.575 90) (size 0.9 0.85) (layers "F.Cu" "F.Paste" "F.Mask") (roundrect_rratio 0.04)
       (net 18 "Net-(D1-RK)") (pinfunction "RK") (pintype "passive"))
@@
   (segment (start 139.75 107.55) (end 139.29 108.9) (width 0.5) (layer "F.Cu") (net 79))
   (segment (start 139.75 107.55) (end 139.4 106.21) (width 0.5) (layer "F.Cu") (net 79))
-  (zone (net 1) (net_name "GND") (layers "F&B.Cu") (hatch edge 0.508)
+  (zone (net 1) (net_name "GND") (layers "F.Cu" "In1.Cu" "In4.Cu" "B.Cu") (hatch edge 0.508)
     (connect_pads yes (clearance 0.2))
     (min_thickness 0.2) (filled_areas_thickness no)
@@
     )
   )
-  (zone (net 3) (net_name "+3V3") (layer "In1.Cu") (hatch edge 0.508)
-    (connect_pads yes (clearance 0.2))
-    (min_thickness 0.2) (filled_areas_thickness no)
-    (fill (thermal_gap 0.508) (thermal_bridge_width 0.508))
-    (polygon
-      (pts
-        (xy 164 115)
-        (xy 136 115)
-        (xy 136 78)
-        (xy 164 78)
-      )
-    )
-  )
   (zone (net 13) (net_name "+BATT") (layer "In2.Cu") (hatch edge 0.508)
     (connect_pads yes (clearance 0.2))
@@
       )
     )
+  )
+  (zone (net 3) (net_name "+3V3") (layer "In3.Cu") (hatch edge 0.508)
+    (connect_pads yes (clearance 0.2))
+    (min_thickness 0.2) (filled_areas_thickness no)
+    (fill (thermal_gap 0.508) (thermal_bridge_width 0.508))
+    (polygon
+      (pts
+        (xy 164 115)
+        (xy 136 115)
+        (xy 136 78)
+        (xy 164 78)
+      )
+    )

Commit message: fix connections and add new ones in schematic
Connections:
- U1 pad 13: /~{GNSS_CS} -> /BATT_MON
- U1 pad 18: unconnected-(U1-PA8-Pad18) -> /~{ACCEL_CS}
- U1 pad 19: unconnected-(U1-PA9-Pad19) -> /~{GNSS_CS}
- U1 pad 2: /MAIN_SENSE -> /LEFT_CTL
- U1 pad 20: /BATT_MON -> /GNSS_PIO
- U1 pad 25: unconnected-(U1-PA15-Pad25) -> /~{GNSS_RESET}
- U1 pad 3: /TAIL_SENSE -> /RADIO_BUSY
- U1 pad 31: GND -> /TAIL_CTL
- U1 pad 5: unconnected-(U1-PA0-Pad5) -> /RADIO_DIO
- U1 pad 6: /TAIL_CTL -> /MAIN_SENSE
- U1 pad 7: /LEFT_CTL -> /~{RADIO_RESET}
- U1 pad 8: /~{RADIO_CS} -> /TAIL_SENSE
- U1 pad 9: /~{ACCEL_CS} -> /~{RADIO_CS}
- U2 pad G4: unconnected-(U2-PIO13/EXTINT-PadG4) -> /GNSS_PIO
- U2 pad J6: unconnected-(U2-RESET_N-PadJ6) -> /~{GNSS_RESET}
- U4 pad 3: unconnected-(U4-~{RESET}-Pad3) -> /~{RADIO_RESET}
- U4 pad 7: unconnected-(U4-BUSY-Pad7) -> /RADIO_BUSY
- U4 pad 8: unconnected-(U4-DIO1-Pad8) -> /RADIO_DIO
